Commit message: replace eef pitch and roll positions

File: urdf/arm_v1.xacro (robot description, xacro)
@@ -22,4 +22,10 @@
     <material name="white">
         <color rgba="1 1 1 1" />
+    </material>
+    <material name="orange">
+        <color rgba="${255/255} ${140/255} ${0/255} 1" />
+    </material>
+    <material name="brown">
+        <color rgba="${139/255} ${69/255} ${19/255} 1" />
     </material>
     <!-- INERTIAL FUNCTIONS -->
@@ -54,5 +60,5 @@
         </inertial>
     </xacro:macro>
-    <!-- MODEL -->
+    <!-- MODEL ARM-->
     <link name="base_link">
         <visual>
@@ -60,5 +66,5 @@
                 <box size="0.15 0.15 0.005"/>
             </geometry>
-            <material name="black"/>
+            <material name="brown"/>
         </visual>
         <collision>
@@ -81,5 +87,5 @@
                 <cylinder radius="0.06" length="0.1"/>
             </geometry>
-            <material name="black"/>
+            <material name="brown"/>
         </visual>
         <collision>
@@ -103,5 +109,5 @@
                 <box size="0.03 0.03 0.3"/>
             </geometry>
-            <material name="yellow"/>
+            <material name="orange"/>
         </visual>
         <collision>
@@ -123,5 +129,5 @@
                 <cylinder radius="0.03" length="0.1"/>
             </geometry>
-            <material name="black"/>
+            <material name="brown"/>
         </visual>
         <collision>
@@ -137,5 +143,5 @@
         <origin xyz="0 0 0.085" rpy="0 0 0"/>
         <axis xyz="1 0 0"/>
-        <limit effort="1000.0" lower="${-3*pi/4}" upper="${3*pi/4}" velocity="0.7"/>
+        <limit effort="1000.0" lower="${-7*pi/8}" upper="${7*pi/8}" velocity="0.7"/>
     </joint>
     <link name="elbow">
@@ -145,5 +151,5 @@
                 <box size="0.03 0.03 0.3"/>
             </geometry>
-            <material name="yellow"/>
+            <material name="orange"/>
         </visual>
         <collision>
@@ -165,5 +171,5 @@
                 <cylinder radius="0.03" length="0.1"/>
             </geometry>
-            <material name="black"/>
+            <material name="brown"/>
         </visual>
         <collision>
@@ -179,5 +185,5 @@
         <origin xyz="0 0 0.085" rpy="0 0 0"/>
         <axis xyz="1 0 0"/>
-        <limit effort="1000.0" lower="${-pi/2}" upper="${pi/2}" velocity="0.7"/>
+        <limit effort="1000.0" lower="${-2*pi/3}" upper="${2*pi/3}" velocity="0.7"/>
     </joint>
     <link name="wrist_pitch">
@@ -187,5 +193,5 @@
                 <box size="0.03 0.03 0.09"/>
             </geometry>
-            <material name="yellow"/>
+            <material name="orange"/>
         </visual>
         <collision>
@@ -207,17 +213,39 @@
                 <cylinder radius="0.03" length="0.1"/>
             </geometry>
-            <material name="black"/>
-        </visual>
-        <collision>
-            <origin xyz="0 0 0.035"/>
-            <geometry>
-                <cylinder radius="0.03" length="0.1"/>
+            <material name="brown"/>
+        </visual>
+        <collision>
+            <origin xyz="0 0 0.035"/>
+            <geometry>
+                <cylinder radius="0.03" length="0.1"/>
+            </geometry>
+        </collision>
+    </link>
+    <joint name="eef_yaw_joint" type="revolute">
+        <parent link="eef_support"/>
+        <child link="eef_yaw"/>
+        <origin xyz="0 0 0.105" rpy="0 0 0"/>
+        <axis xyz="0 1 0"/>
+        <limit effort="1000.0" lower="${-pi/4}" upper="${pi/4}" velocity="0.7"/>
+    </joint>
+    <link name="eef_yaw">
+        <visual>
+            <origin xyz="0 0 0"  rpy="0 ${pi/2} ${pi/2}"/>
+            <geometry>
+                <cylinder radius="0.02" length="0.08"/>
+            </geometry>
+            <material name="brown"/>
+        </visual>
+        <collision>
+            <origin xyz="0 0 0" rpy="0 ${pi/2} ${pi/2}"/>
+            <geometry>
+                <cylinder radius="0.02" length="0.08"/>
             </geometry>
         </collision>
     </link>
     <joint name="eef_roll_joint" type="revolute">
-        <parent link="eef_support"/>
+        <parent link="eef_yaw"/>
         <child link="eef_roll"/>
-        <origin xyz="0 0 0.085" rpy="0 0 0"/>
+        <origin xyz="0 0 0.02" rpy="0 0 0"/>
         <axis xyz="0 0 1"/>
         <limit effort="1000.0" lower="${-pi}" upper="${pi}" velocity="0.7"/>
@@ -229,5 +257,5 @@
                 <cylinder radius="0.05" length="0.005"/>
             </geometry>
-            <material name="yellow"/>
+            <material name="orange"/>
         </visual>
         <collision>
@@ -238,50 +266,22 @@
         </collision>
     </link>
-    <joint name="eef_pitch_joint" type="revolute">
+    <joint name="safety_link_joint" type="fixed">
         <parent link="eef_roll"/>
-        <child link="eef_pitch"/>
-        <origin xyz="0 0 0.025" rpy="0 0 0"/>
-        <axis xyz="1 0 0"/>
-        <limit effort="1000.0" lower="${-pi/4}" upper="${pi/4}" velocity="0.7"/>
-    </joint>
-    <link name="eef_pitch">
-        <visual>
-            <origin xyz="0 0 0"  rpy="0 ${pi/2} 0"/>
-            <geometry>
-                <cylinder radius="0.02" length="0.08"/>
-            </geometry>
-            <material name="black"/>
-        </visual>
-        <collision>
-            <origin xyz="0 0 0" rpy="0 ${pi/2} 0"/>
-            <geometry>
-                <cylinder radius="0.02" length="0.08"/>
-            </geometry>
-        </collision>
-    </link>
-    <joint name="gripper_attacher_joint" type="fixed">
-        <parent link="eef_pitch"/>
-        <child link="gripper_attacher"/>
-        <origin xyz="0 0 0.02" rpy="0 0 0"/>
-    </joint>
-    <link name="gripper_attacher">
-        <visual>
-            <origin xyz="0 0 0.005"/>
-            <geometry>
-                <box size="0.1 0.075 0.01"/>
-            </geometry>
-            <material name="white"/>
-        </visual>
-        <collision>
-            <origin xyz="0 0 0.005"/>
-            <geometry>
-                <box size="0.1 0.075 0.01"/>
-            </geometry>
-        </collision>
-    </link>
+        <child link="safety_link"/>
+        <origin xyz="0 0 0.005" rpy="0 0 0"/>
+    </joint>
+    <link name="safety_link">
+        <collision>
+            <origin xyz="0 0 0"/>
+            <geometry>
+                <sphere radius="0.03"/>
+            </geometry>
+        </collision>
+    </link>
+    <!-- MODEL GRIPPER -->
     <joint name="gripper_support_joint" type="fixed">
-        <parent link="gripper_attacher"/>
+        <parent link="safety_link"/>
         <child link="gripper_support"/>
-        <origin xyz="0 0 0.01" rpy="0 0 0"/>
+        <origin xyz="0 0 0" rpy="0 0 0"/>
     </joint>
     <link name="gripper_support">

Commit message: move fingers up to avoid collision

File: urdf/arm_v1.xacro (robot description, xacro)
@@ -309,5 +309,5 @@
     <link name="gripper_leftfinger">
         <visual>
-            <origin xyz="0 0 0.04"/>
+            <origin xyz="0 0 0.05"/>
             <geometry>
                 <box size="0.02 0.02 0.1"/>
@@ -316,5 +316,5 @@
         </visual>
         <collision>
-            <origin xyz="0 0 0.04"/>
+            <origin xyz="0 0 0.05"/>
             <geometry>
                 <box size="0.02 0.02 0.1"/>
@@ -331,5 +331,5 @@
     <link name="gripper_rightfinger">
         <visual>
-            <origin xyz="0 0 0.04"/>
+            <origin xyz="0 0 0.05"/>
             <geometry>
                 <box size="0.02 0.02 0.1"/>
@@ -338,5 +338,5 @@
         </visual>
         <collision>
-            <origin xyz="0 0 0.04"/>
+            <origin xyz="0 0 0.05"/>
             <geometry>
                 <box size="0.02 0.02 0.1"/>
